File: Nano_Lambda.sch (KiCad schematic (older format))
At the start: 70 parts, among them IC1 LMV321?M5, IC2 LM4041DBZ, J1 +12_IN, J10 PD3, J11 GP3, J12 DAC1, J13 DAC2, J14 Out1, J2 GND, J3 +12V_NL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

Commit message: Change to Version 0.9b
Changed wrong CJ125 Footprint to Footprint with 0.8mm pitch.
Parts:
- U1: footprint Housings_QFP:LQFP-32_5x5mm_Pitch0.5mm -> Housings_QFP:LQFP-32_7x7mm_Pitch0.8mm
Changed lines of the file:
@@
 F 0 "U1" H 3500 2686 59  0000 C CNN
 F 1 "CJ125_32" H 3500 2581 59  0000 C CNN
-F 2 "Housings_QFP:LQFP-32_5x5mm_Pitch0.5mm" H 3500 2000 50  0001 C CNN
+F 2 "Housings_QFP:LQFP-32_7x7mm_Pitch0.8mm" H 3500 2000 50  0001 C CNN
 F 3 "" H 3500 2000 50  0001 C CNN
 	1    3500 2000
